Commit message: added esp32 launch file and fixes to urdf

File: linorobot2_description/urdf/2wd_properties.urdf.xacro (robot description, xacro)
@@ -1,19 +1,19 @@
 <?xml version="1.0"?>
 <robot xmlns:xacro="http://ros.org/wiki/xacro">
-  <xacro:property name="base_length" value="0.24" />
-  <xacro:property name="base_width" value="0.275" />
+  <xacro:property name="base_length" value="0.17" />
+  <xacro:property name="base_width" value="0.126" />
   <xacro:property name="base_height" value="0.003" />
   <xacro:property name="base_mass" value="1" />
-  <xacro:property name="wheel_radius" value="0.045" />
-  <xacro:property name="wheel_width" value="0.01" />
-  <xacro:property name="wheel_pos_x" value="0.0" />
-  <xacro:property name="wheel_pos_y" value="0.13" />
+  <xacro:property name="wheel_radius" value="0.03375" />
+  <xacro:property name="wheel_width" value="0.0261" />
+  <xacro:property name="wheel_pos_x" value="0.06" />
+  <xacro:property name="wheel_pos_y" value="0.063" />
   <xacro:property name="wheel_pos_z" value="-0.03" />
   <xacro:property name="wheel_mass" value=".1" />
   <xacro:property name="wheel_torque" value="20" />
-  <xacro:property name="front_caster_wheel" value="true" />
+  <xacro:property name="front_caster_wheel" value="false" />
   <xacro:property name="rear_caster_wheel" value="true" />
   <xacro:property name="laser_pose">
-    <origin xyz="0.12 0 0.33" rpy="0 0 0"/>
+    <origin xyz="0.06 0 0.10" rpy="0 0 0"/>
   </xacro:property>
   <xacro:property name="depth_sensor_pose">

File: linorobot2_description/urdf/robots/2wd.urdf.xacro (robot description, xacro)
@@ -57,7 +57,7 @@
     <xacro:insert_block name="laser_pose" />
   </xacro:generic_laser>
-  <xacro:depth_sensor>
+  <!-- <xacro:depth_sensor>
     <xacro:insert_block name="depth_sensor_pose" />
-  </xacro:depth_sensor>
+  </xacro:depth_sensor> -->
   <xacro:diff_drive_controller
     wheel_separation="${wheel_pos_y * 2}"
